Commit message: working rviz model

File: acrobot_description/acrobot/robot.urdf (robot description, URDF)
Before this commit: robot acrobot, 3 links, 2 joints
Links:
- link part_1: geometry collision mesh filename=package://acrobot_description/acrobot/assets/part_1.stl; collision mesh filename=package://acrobot_description/acrobot/assets/part_1__2.stl
- link part_1_2: geometry collision mesh filename=package://acrobot_description/acrobot/assets/part_1__2.stl; collision mesh filename=package://acrobot_description/acrobot/assets/part_1__3.stl
- link part_1_3: geometry collision mesh filename=package://acrobot_description/acrobot/assets/part_1__4.stl; visual mesh filename=package://acrobot_description/acrobot/assets/part_1__4.stl
